File: RemoteController/RemoteController.kicad_pcb (KiCad board)
At the start: 2 copper layers, 66.8 x 142.2 mm, 35 parts, among them J1 SSD1306, J2 Conn_01x02_Male, J3 Conn_01x02_Male, J4 Conn_01x02_Male, J5 Conn_01x06_Male, SW1 RotaryEncoder_Switch, SW2 SW_Push_SPDT, SW3 SW_Push_SPDT, SW4 SW_Push_SPDT, SW5 SW_Push_SPDT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

Commit message: Fix Remote PCB for future version
Parts:
- added R3: 10k, Resistor_THT:R_Axial_DIN0207_L6.3mm_D2.5mm_P10.16mm_Horizontal, B.Cu at (155.7, 151.1)
- added RN5: 10k, Resistor_THT:R_Array_SIP6, B.Cu at (154.3, 147.8)
- moved C3 27.7 mm to (146.8, 76.2)
- moved J3 2.15 mm to (159.9, 146.3)
- moved R1 0.13 mm to (149.6, 63.4)
Routing:
- net +3V3: track 295.1 -> 332.0 mm
- net /L1: track 44.8 -> 70.2 mm
- net /L4: track 29.5 -> 51.5 mm
- net GND: track 62.6 -> 79.1 mm
- net /L3: track 30.9 -> 41.2 mm
- net /L2: track 43.6 -> 49.9 mm
- net /P5_R: track 126.8 -> 121.1 mm
- net /UNUSED_GPIO2: track 19.5 -> 22.8 mm
- net /VIN_MCU: track 165.6 -> 163.4 mm
Other:
- board text added: "Train remote V2 09/2023"
- board text removed: "Train remote V1 09/2023"
