File: RemoteController/RemoteController.kicad_sch (KiCad schematic)
At the start: 35 parts, among them J1 SSD1306, J2 Conn_01x02_Male, J3 Conn_01x02_Male, J4 Conn_01x02_Male, J5 Conn_01x06_Male, SW1 RotaryEncoder_Switch, SW2 SW_Push_SPDT, SW3 SW_Push_SPDT, SW4 SW_Push_SPDT, SW5 SW_Push_SPDT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

Commit message: Fix Remote PCB for future version
Parts:
- added R?: 10k, Resistor_THT:R_Axial_DIN0207_L6.3mm_D2.5mm_P10.16mm_Horizontal, symbol Device:R
- added RN?: 10k, Resistor_THT:R_Array_SIP6, symbol Device:R_Pack03_SIP
Connections:
- net GND: now also R?.1, RN?.2 (R1.2), RN?.4 (R2.2), RN?.6 (R3.2)
- net L1: now also RN?.1 (R1.1)
- net L2: now also RN?.3 (R2.1)
- net L3: now also RN?.5 (R3.1)
- net L4: now also R?.2
Changed lines of the file:
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@@
+    (stroke (width 0) (type default) (color 0 0 0 0))
+  )
+  (wire (pts (xy 142.875 87.63) (xy 140.335 87.63))
     (stroke (width 0) (type default) (color 0 0 0 0))
   )
@@
     (stroke (width 0) (type default) (color 0 0 0 0))
   )
+  (wire (pts (xy 142.875 95.25) (xy 142.875 87.63))
+    (stroke (width 0) (type default) (color 0 0 0 0))
+  )
   (wire (pts (xy 140.335 160.02) (xy 153.035 160.02))
     (stroke (width 0) (type default) (color 0 0 0 0))
@@
     (effects (font (size 1.27 1.27)) (justify right bottom))
   )
+  (label "L1" (at 114.935 95.885 270)
+    (effects (font (size 1.27 1.27)) (justify right bottom))
+  )
   (label "P1_R" (at 37.465 122.555 0)
     (effects (font (size 1.27 1.27)) (justify left bottom))
@@
     (effects (font (size 1.27 1.27)) (justify right bottom))
   )
+  (label "L4" (at 140.335 95.25 270)
+    (effects (font (size 1.27 1.27)) (justify right bottom))
+  )
   (label "UNUSED_GPIO16" (at 141.605 65.405 180)
     (effects (font (size 1.27 1.27)) (justify right bottom))
@@
     (effects (font (size 1.27 1.27)) (justify right bottom))
   )
+  (label "L2" (at 122.555 95.885 270)
+    (effects (font (size 1.27 1.27)) (justify right bottom))
+  )
   (label "P5_L" (at 140.335 121.92 180)
     (effects (font (size 1.27 1.27)) (justify right bottom))
@@
     (effects (font (size 1.27 1.27)) (justify right bottom))
   )
+  (label "P5_R" (at 102.235 95.885 270)
+    (effects (font (size 1.27 1.27)) (justify right bottom))
+  )
   (label "P4_L" (at 37.465 154.94 0)
     (effects (font (size 1.27 1.27)) (justify left bottom))
@@
     (effects (font (size 1.27 1.27)) (justify left bottom))
   )
+  (label "L3" (at 130.175 95.885 270)
+    (effects (font (size 1.27 1.27)) (justify right bottom))
+  )
   (label "L4" (at 140.335 134.62 180)
-    (effects (font (size 1.27 1.27)) (justify right bottom))
-  )
-  (label "P5_R" (at 102.235 95.885 270)
     (effects (font (size 1.27 1.27)) (justify right bottom))
   )
@@
     )
     (property "Datasheet" "~" (id 3) (at 163.83 111.76 0)
+      (effects (font (size 1.27 1.27)) hide)
+    )
+    (pin "1")
+    (pin "2")
+  )
+  (symbol (lib_id "Device:R") (at 140.335 91.44 0) (unit 1)
+    (in_bom yes) (on_board yes) (fields_autoplaced)
+    (property "Reference" "R?" (id 0) (at 142.24 90.1699 0)
+      (effects (font (size 1.27 1.27)) (justify left))
+    )
+    (property "Value" "10k" (id 1) (at 142.24 92.7099 0)
+      (effects (font (size 1.27 1.27)) (justify left))
+    )
+    (property "Footprint" "Resistor_THT:R_Axial_DIN0207_L6.3mm_D2.5mm_P10.16mm_Horizontal" (id 2) (at 138.557 91.44 90)
+      (effects (font (size 1.27 1.27)) hide)
+    )
+    (property "Datasheet" "~" (id 3) (at 140.335 91.44 0)
       (effects (font (size 1.27 1.27)) hide)
     )
@@
     )
     (pin "1")
+  )
+  (symbol (lib_id "Device:R_Pack03_SIP") (at 122.555 90.805 0) (unit 1)
+    (in_bom yes) (on_board yes) (fields_autoplaced)
+    (property "Reference" "RN?" (id 0) (at 123.825 81.28 0))
+    (property "Value" "10k" (id 1) (at 123.825 83.82 0))
+    (property "Footprint" "Resistor_THT:R_Array_SIP6" (id 2) (at 137.16 90.805 90)
+      (effects (font (size 1.27 1.27)) hide)
+    )
+    (property "Datasheet" "http://www.vishay.com/docs/31509/csc.pdf" (id 3) (at 122.555 90.805 0)
+      (effects (font (size 1.27 1.27)) hide)
+    )
+    (pin "1")
+    (pin "2")
+    (pin "3")
+    (pin "4")
+    (pin "5")
+    (pin "6")
   )
   (symbol (lib_id "power:GND") (at 254.635 40.005 0) (unit 1)
@@
     (pin "1")
   )
-  (symbol (lib_id "power:GND") (at 104.775 95.885 0) (unit 1)
-    (in_bom yes) (on_board yes) (fields_autoplaced)
-    (property "Reference" "#PWR0122" (id 0) (at 104.775 102.235 0)
-      (effects (font (size 1.27 1.27)) hide)
-    )
-    (property "Value" "GND" (id 1) (at 104.775 100.33 0))
-    (property "Footprint" "" (id 2) (at 104.775 95.885 0)
-      (effects (font (size 1.27 1.27)) hide)
-    )
-    (property "Datasheet" "" (id 3) (at 104.775 95.885 0)
+  (symbol (lib_id "power:GND") (at 142.875 95.25 0) (unit 1)
+    (in_bom yes) (on_board yes) (fields_autoplaced)
+    (property "Reference" "#PWR0136" (id 0) (at 142.875 101.6 0)
+      (effects (font (size 1.27 1.27)) hide)
+    )
+    (property "Value" "GND" (id 1) (at 142.875 99.695 0))
+    (property "Footprint" "" (id 2) (at 142.875 95.25 0)
+      (effects (font (size 1.27 1.27)) hide)
+    )
+    (property "Datasheet" "" (id 3) (at 142.875 95.25 0)
       (effects (font (size 1.27 1.27)) hide)
     )
@@
     (pin "1")
   )
+  (symbol (lib_id "power:GND") (at 117.475 95.885 0) (unit 1)
+    (in_bom yes) (on_board yes) (fields_autoplaced)
+    (property "Reference" "#PWR?" (id 0) (at 117.475 102.235 0)
+      (effects (font (size 1.27 1.27)) hide)
+    )
+    (property "Value" "GND" (id 1) (at 117.475 100.33 0))
+    (property "Footprint" "" (id 2) (at 117.475 95.885 0)
+      (effects (font (size 1.27 1.27)) hide)
+    )
+    (property "Datasheet" "" (id 3) (at 117.475 95.885 0)
+      (effects (font (size 1.27 1.27)) hide)
+    )
+    (pin "1")
+  )
   (symbol (lib_id "Mechanical:MountingHole") (at 234.315 119.38 0) (unit 1)
     (in_bom yes) (on_board yes) (fields_autoplaced)
@@
     )
   )
+  (symbol (lib_id "power:GND") (at 125.095 95.885 0) (unit 1)
+    (in_bom yes) (on_board yes) (fields_autoplaced)
+    (property "Reference" "#PWR?" (id 0) (at 125.095 102.235 0)
+      (effects (font (size 1.27 1.27)) hide)
+    )
+    (property "Value" "GND" (id 1) (at 125.095 100.33 0))
+    (property "Footprint" "" (id 2) (at 125.095 95.885 0)
+      (effects (font (size 1.27 1.27)) hide)
+    )
+    (property "Datasheet" "" (id 3) (at 125.095 95.885 0)
+      (effects (font (size 1.27 1.27)) hide)
+    )
+    (pin "1")
+  )
   (symbol (lib_id "Device:R") (at 142.24 24.13 90) (unit 1)
     (in_bom yes) (on_board yes) (fields_autoplaced)
@@
     )
     (property "Datasheet" "" (id 3) (at 153.035 111.76 0)
+      (effects (font (size 1.27 1.27)) hide)
+    )
+    (pin "1")
+  )
+  (symbol (lib_id "power:GND") (at 132.715 95.885 0) (unit 1)
+    (in_bom yes) (on_board yes) (fields_autoplaced)
+    (property "Reference" "#PWR?" (id 0) (at 132.715 102.235 0)
+      (effects (font (size 1.27 1.27)) hide)
+    )
+    (property "Value" "GND" (id 1) (at 132.715 100.33 0))
+    (property "Footprint" "" (id 2) (at 132.715 95.885 0)
+      (effects (font (size 1.27 1.27)) hide)
+    )
+    (property "Datasheet" "" (id 3) (at 132.715 95.885 0)
       (effects (font (size 1.27 1.27)) hide)
     )
@@
     (pin "6")
   )
+  (symbol (lib_id "power:GND") (at 104.775 95.885 0) (unit 1)
+    (in_bom yes) (on_board yes) (fields_autoplaced)
+    (property "Reference" "#PWR?" (id 0) (at 104.775 102.235 0)
+      (effects (font (size 1.27 1.27)) hide)
+    )
+    (property "Value" "GND" (id 1) (at 104.775 100.33 0))
+    (property "Footprint" "" (id 2) (at 104.775 95.885 0)
+      (effects (font (size 1.27 1.27)) hide)
+    )
+    (property "Datasheet" "" (id 3) (at 104.775 95.885 0)
+      (effects (font (size 1.27 1.27)) hide)
+    )
+    (pin "1")
+  )
   (symbol (lib_id "power:GND") (at 131.445 24.13 0) (mirror y) (unit 1)
     (in_bom yes) (on_board yes) (fields_autoplaced)
@@
       (reference "#PWR0121") (unit 1) (value "GND") (footprint "")
     )
-    (path "/6618d3da-1e03-4d0e-a396-a1cd1565b6d5"
-      (reference "#PWR0122") (unit 1) (value "GND") (footprint "")
-    )
     (path "/a522174e-9954-45a8-baea-5cedf5574903"
       (reference "#PWR0123") (unit 1) (value "GND") (footprint "")
@@
       (reference "#PWR0135") (unit 1) (value "GND") (footprint "")
     )
+    (path "/67803602-03b0-4afe-b6c4-a15f67c52d8f"
+      (reference "#PWR0136") (unit 1) (value "GND") (footprint "")
+    )
     (path "/d5c50fbb-0351-4dbb-ad23-4f49511605b9"
       (reference "#PWR0137") (unit 1) (value "GND") (footprint "")
     )
+    (path "/8e7569e6-06a7-479b-b2fa-dda44924f561"
+      (reference "#PWR?") (unit 1) (value "GND") (footprint "")
+    )
+    (path "/9fe7d040-5c24-4118-9afb-4ba3cd0abd7b"
+      (reference "#PWR?") (unit 1) (value "GND") (footprint "")
+    )
+    (path "/aadc3ee9-2fd5-4115-9add-f58cf18c279f"
+      (reference "#PWR?") (unit 1) (value "GND") (footprint "")
+    )
+    (path "/d37170e9-5807-4fef-9aa9-1828e0e73293"
+      (reference "#PWR?") (unit 1) (value "GND") (footprint "")
+    )
     (path "/6a8dca6d-426e-4119-872a-ae71c6883aa6"
       (reference "C1") (unit 1) (value "0.1uF") (footprint "Capacitor_THT:CP_Radial_D4.0mm_P2.00mm")
@@
       (reference "R2") (unit 1) (value "R") (footprint "Resistor_THT:R_Axial_DIN0207_L6.3mm_D2.5mm_P10.16mm_Horizontal")
     )
+    (path "/049da9cd-5423-4560-b9ed-b4ac5e24bc8e"
+      (reference "R?") (unit 1) (value "10k") (footprint "Resistor_THT:R_Axial_DIN0207_L6.3mm_D2.5mm_P10.16mm_Horizontal")
+    )
     (path "/ec3ed3a4-6b37-4fa0-876d-a3fed51f9a09"
       (reference "RN1") (unit 1) (value "10k") (footprint "Resistor_THT:R_Array_SIP6")
@@
       (reference "RN4") (unit 1) (value "10k") (footprint "Resistor_THT:R_Array_SIP6")
     )
+    (path "/1f63fd73-b7ee-489a-8ec3-2501312312bf"
+      (reference "RN?") (unit 1) (value "10k") (footprint "Resistor_THT:R_Array_SIP6")
+    )
     (path "/b7efde0b-779c-44e8-8352-f6b887153b57"
